File: H07R80/Design/H07R8.sch (EAGLE design)
At the start: 17 parts, among them P2 HEXABIT_X2_P1_P5_EDIT_POWER_P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, U1 STM32G0B1CEU6N, X1 XTALL_CSTCE8M00G52

Commit message: - The reviewed version is complete.
Parts:
- removed JP1: R, HEXABITZ_USER_INTERFACE_PARTS:PINHD-1X1
- removed JP2: (no value), pinhead:PINHD-1X3
- removed P2: HEXABIT_X2_P1_P5_EDIT_POWER_PADS, hexabitz_connectors:HEXABIT_X2_P1_P5_EDIT_POWER_PADS
- added +1.8V, GND: PAD4, HEXABITZ_CONNECTION_PARTS:PAD4
- added C10, C11, C18, C19, C20, C22, C23, C24, C25, C27, C28, C39, C40: 0.47uF, HEXABITZ_RCLS:C-0603
- added C12, C15, C16, C17, C33, C34, C35, C36, C37, C44: 1uF, HEXABITZ_RCLS:C-0603
- added C13, C45, C8, C9: 100nF, HEXABITZ_RCLS:C-0603
- added C14: 2.2uF, HEXABITZ_RCLS:C-0603
- added C21: 0.01uF, HEXABITZ_RCLS:C-0603
- added C29, C41: DNP, HEXABITZ_RCLS:C-0603
- added C30, C31: 47uF, HEXABITZ_RCLS:A780EN476M1HLAS050
- added C32, C38, C42, C43: 100pF, HEXABITZ_RCLS:C-0603
- added FB3, FB4, FB5, FB6: SHORT(0Ohm), HEXABITZ_RCLS:FB-0603
- added J1, J2, J3: 1751248PHOENIX_CONTACT_1751248_0_0, hexabitz_connectors:1751248PHOENIX_CONTACT_1751248_0_0
- added J4: SJ-3524-SMT-TR, HEXABITZ_ICs:SJ-3524-SMT-TRU
- added P1: HEXABIT_X3_ROW_NO_P4_P6_P7_P8_P10_P14, hexabitz_connectors:HEXABIT_X3_ROW_NO_P4_P6_P7_P8_P10_P14
- added Q2: AO3400AALPHA_&_OMEGA_SEMICONDUCTOR_AO3400A_0_0, HEXABITZ_ICs:AO3400AALPHA_&_OMEGA_SEMICONDUCTOR_AO3400A_0_0
- added R: (no value), HEXABITZ_USER_INTERFACE_PARTS:PINHD-1X1
- added R10, R11, R12, R13, R14, R5: 100, HEXABITZ_RCLS:R-0603
- added R4: 100K, HEXABITZ_RCLS:R-0603
- added R6, R9: 10K, HEXABITZ_RCLS:R-0603
- added R7, R8: 4.7K, HEXABITZ_RCLS:R-0603
- added SWD: (no value), pinhead:PINHD-1X3
- added U2: MAX9867ETJ+T, HEXABITZ_ICs:MAX9867ETJ+T
- added U3: TS3A44159RGTRTEXAS_INSTRUMENTS_TS3A44159RGTR_0_0, HEXABITZ_ICs:TS3A44159RGTRTEXAS_INSTRUMENTS_TS3A44159RGTR_0_0
- added U5: MAX9704ETJ+, HEXABITZ_ICs:MAX9704ETJ+
- added U6: MIC5365-1.8YD5-TRMICROCHIP_MIC5365-1_8YD5-TR_0_0, HEXABITZ_ICs:MIC5365-1.8YD5-TRMICROCHIP_MIC5365-1_8YD5-TR_0_0
- C1: CAPACITANCE (none) -> 100nF; MFN (none) -> AVX CORPORATION; MPN (none) -> 0603YC104K4T2A; OCTOPART_URL (none) -> 'https://octopart.com/0603yc104k4t2a-avx+interconnect+%2F+e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; TOLERANCE (none) -> 10%; VOLTAGE_RATING (none) -> 16.0 V
- C2: value 4.7uF -> 100nF; device HEXABITZ_RCLS:C-0805-POL -> HEXABITZ_RCLS:C-0603; CAPACITANCE (none) -> 100nF; MFN (none) -> AVX CORPORATION; MPN (none) -> '0603YC104K4T2A; OCTOPART_URL (none) -> 'https://octopart.com/0603yc104k4t2a-avx+interconnect+%2F+e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; TOLERANCE (none) -> 10%; VOLTAGE_RATING (none) -> 16.0 V
- C3: value 100nF -> 4.7uF; device HEXABITZ_RCLS:C-0603 -> HEXABITZ_RCLS:C-0805-POL; CAPACITANCE (none) -> 4.7uF; MFN (none) -> 'Panasonic; MPN (none) -> '10TPU4R7MSI; OCTOPART_URL (none) -> https://octopart.com/10tpu4r7msi-panasonic-29487748?r=sp; TOLERANCE (none) -> 20%; VOLTAGE_RATING (none) -> 10.0 V
- C4: value 1uF -> 100nF; device HEXABITZ_RCLS:C-0805-POL -> HEXABITZ_RCLS:C-0603; CAPACITANCE (none) -> 100nF; MFN (none) -> AVX CORPORATION; MPN (none) -> '0603YC104K4T2A; OCTOPART_URL (none) -> 'https://octopart.com/0603yc104k4t2a-avx+interconnect+%2F+e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; TOLERANCE (none) -> 10%; VOLTAGE_RATING (none) -> 16.0 V
- C5: value 100nF -> 1uF; device HEXABITZ_RCLS:C-0603 -> HEXABITZ_RCLS:C-0805-POL; CAPACITANCE (none) -> 4.7uF; MFN (none) -> 'YAGEO [VA]; MPN (none) -> 'CC0805KKX7R7BB105; OCTOPART_URL (none) -> 'https://octopart.com/cc0805kkx7r7bb105-yageo-8376555?r=sp; TOLERANCE (none) -> 20%; VOLTAGE_RATING (none) -> 10.0 V
- C6: CAPACITANCE (none) -> 100nF; MFN (none) -> AVX CORPORATION; MPN (none) -> '0603YC104K4T2A; OCTOPART_URL (none) -> 'https://octopart.com/0603yc104k4t2a-avx+interconnect+%2F+e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; TOLERANCE (none) -> 10%; VOLTAGE_RATING (none) -> 16.0 V
- C7: CAPACITANCE (none) -> 1.00uF; MFN (none) -> 'Panasonic; MPN (none) -> '10TPU4R7MSI; OCTOPART_URL (none) -> https://octopart.com/10tpu4r7msi-panasonic-29487748?r=sp; TOLERANCE (none) -> 10%; VOLTAGE_RATING (none) -> 16.0 V
- D1: device Hexabitz:VLMS1300-GS08 -> HEXABITZ_USER_INTERFACE_PARTS:VLMS1300-GS08; MFN Vishay -> (none); MPN VLMS1300-GS08 -> (none); OCTOPART_URL https://octopart.com/vlms1300-gs08-vishay-21709201?r=sp&s=_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 -> (none)
- FB1: device HEXABITZ_RCLS:FB-0603 -> HEXABITZ_RCLS:FB-TDK_MMZ1608Y300B; MFN (none) -> TDK; MPN (none) -> MMZ1608Y300BTA00; OCTOPART_URL (none) -> https://octopart.com/mmz1608y300bta00-tdk-7906990?r=sp
- R1: value 10K -> 0.0R; MFN (none) -> YAGEO [VR]; MPN (none) -> RC0603JR-070RL; OCTOPART_URL (none) -> https://octopart.com/rc0603jr-070rl-yageo-1241539?r=sp; RESISTANCE (none) -> 0R
- R2: value 0.0R -> 270R; MFN (none) -> 'Panasonic; MPN (none) -> 'ERJ-3GEYJ271V; OCTOPART_URL (none) -> https://octopart.com/erj-3geyj271v-panasonic-55560546?r=sp; RESISTANCE (none) -> 270R
- R3: value 270R -> 10K; MFN (none) -> Vishay; MPN (none) -> '060300J0103T5E; OCTOPART_URL (none) -> https://octopart.com/search?q=060300J0103T5E&currency=USD&s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; RESISTANCE (none) -> 10K
- X1: value XTALL_CSTCE8M00G52 -> 8MHZ; device Hexabitz:XTALL_CSTCE8M00G52 -> HEXABITZ_OTHER_PARTS:XTALL_CSTCE8M00G52; MPN (none) -> CSTNE8M00G550000R0; OCTOPART_URL (none) -> https://octopart.com/cstne8m00g550000r0-murata-91406934?r=sp
Connections:
- removed net CLK: JP2.1, JP2.2, R1.2, U1.PA14-BOOT0
- removed net DATA: JP2.3, U1.PA13
- removed net VSSA: C1.2, C2.-, C3.2, C4.-, R2.1, U1.VSS/VSSA
- new net +1.8V: +1.8V.P$1, C17.2, C33.2, C35.2, C36.2, U2.AVDD, U2.DVDD, U2.PVDD, U6.VOUT
- new net +12V: C12.1, C30.+, C31.+, C8.1, C9.2, J1.1, U5.VDD@1, U5.VDD@2, U5.VDD@3, U5.VDD@4
- new net AUDIO_JACK_IN_L: C19.1, J4.2, R9.1
- new net AUDIO_JACK_IN_R: C27.1, J4.3
- new net C: R3.2, SWD.1, SWD.2, U1.PA14-BOOT0
- new net CODEC_IRQN_OUT: R6.1, U1.PB1, U2.!IRQ
- new net CODEC_LOUT_N: C32.2, FB5.1, U2.LOUTN
- new net CODEC_LOUT_P: C38.2, FB4.1, U2.LOUTP
- new net CODEC_ROUT_N: C42.2, FB6.1, U2.ROUTN
- new net CODEC_ROUT_P: C43.2, FB3.1, U2.ROUTP
- new net D: SWD.3, U1.PA13
- new net DC_JACK_DETECT: J4.4, R4.2, U3.IN1-2, U3.IN3-4
- new net GND1: C10.1, C14.1, C15.1, C16.1, C17.1, C2.1, C20.2, C21.2, C28.1, C3.-, C30.-, C31.-, C32.1, C33.1, C34.1, C35.1, C36.1, C37.1, C38.1, C4.1, C42.1, C43.1, C44.1, C45.2, C5.-, C8.2, C9.1, GND.P$1, J1.2, J4.1, Q2.S, R1.2, R4.1, U1.VSS/VSSA, U2.AGND, U2.DGND, U2.EP, U2.PGND, U3.EP, U3.GND, U5.AGND@1, U5.EP, U5.PGND@1, U5.PGND@2, U5.PGND@3, U5.PGND@4, U6.GND
- new net I2C_SCL: R7.2, U1.PB13, U2.SCL
- new net I2C_SDA: R8.2, U1.PB14, U2.SDA
- new net I2S_CLK: U1.PA5, U2.BCLK
- new net I2S_MCK: U1.PA6, U2.MCLK
- new net I2S_SD: U1.PA7, U2.SDIN
- new net I2S_WS: U1.PA4, U2.LRCLK
- new net N$10: C13.1, U5.C1P
- new net N$11: C39.2, U3.NO3
- new net N$12: C1.2, R.1, U1.PF2-NRST
- new net N$13: C40.2, U3.NO4
- new net N$14: C19.2, U3.NC1
- new net N$15: C13.2, U5.C1N
- new net N$17: C27.2, U3.NC3
- new net N$18: C22.1, C29.2, FB4.2
- new net N$19: C23.1, C29.1, FB5.2
- new net N$20: C39.1, C41.2, FB3.2
- new net N$21: C10.2, U3.NC2
- new net N$22: C28.2, U3.NC4
- new net N$23: C16.2, U2.REG
- new net N$24: C14.2, U2.REF
- new net N$25: C34.2, U2.PREG
- new net N$26: C11.2, U5.INL+
- new net N$27: C11.1, U3.COM1
- new net N$28: C18.1, U3.COM2
- new net N$29: C24.1, U3.COM3
- new net N$3: R2.2, U1.PA12[PA10]
- new net N$30: C25.1, U3.COM4
- new net N$33: C18.2, U5.INL-
- new net N$34: C24.2, U5.INR+
- new net N$35: C15.2, U2.MICBIAS
- new net N$36: C20.1, Q2.D, U5.SS
- new net N$37: C25.2, U5.INR-
- new net N$39: R13.1, U5.FS1
- new net N$4: D1.A, R2.1
- new net N$40: R14.1, U5.FS2
- new net N$41: R12.1, U5.!SHDN!
- new net N$42: R11.1, U5.G1
- new net N$43: R10.1, U5.G2
- new net N$44: Q2.G, R5.1
- new net N$45: U1.PA11[PA9]
- new net N$7: C12.2, U5.CHOLD
- new net N$9: C23.2, U3.NO2
- new net OUTL+: J2.2, U5.OUTL+@1, U5.OUTL+@2
- new net OUTL-: J2.1, U5.OUTL-@1, U5.OUTL-@2
- new net OUTR+: J3.2, U5.OUTR+@1, U5.OUTR+@2
- new net OUTR-: J3.1, U5.OUTR-@1, U5.OUTR-@2
- new net PWR_AMP_FSEL1: R13.2, U1.PB4
- new net PWR_AMP_FSEL2: R14.2, U1.PB3
- new net PWR_AMP_GAIN1: R11.2, U1.PB6
- new net PWR_AMP_GAIN2: R10.2, U1.PB5
- new net PWR_AMP_MUTE: R5.2, U1.PD1
- new net PWR_AMP_SHDN: R12.2, U1.PB7
- new net USART4_RX: P1.SD11, U1.PA1
- new net USART4_TX: P1.SU11, U1.PA0
- net GND: now also C1.1, C6.1, P1.GND1, P1.GND10, P1.GND11, P1.GND12, P1.GND13, P1.GND2, P1.GND3, P1.GND4, P1.GND5, P1.GND6, R3.1; no longer C5.2, C6.2, P2.GND1, P2.GND2, P2.GND3, P2.GND4, P2.GND5, P2.GND6, P2.GND7, P2.GND8, R2.2
- net N$1: now also U1.PF0-OSC_IN, X1.1; no longer D1.A, R3.2
- net N$2: now also U1.PF1-OSC_OUT, X1.3; no longer R3.1, U1.PB7
- net N$5: now also C40.1, C41.1, FB6.2; no longer U1.PF1-OSC_OUT, X1.1
- net N$6: now also C21.1, U5.REG; no longer U1.PF0-OSC_IN, X1.3
- net N$8: now also C22.2, U3.NO1; no longer C6.1, JP1.1, U1.PF2-NRST
- net USART1_RX: now also P1.SD1; no longer P2.SD4
- net USART1_TX: now also P1.SU1; no longer P2.SU4
- net USART2_RX: now also P1.SD2; no longer P2.SD2
- net USART2_TX: now also P1.SU2; no longer P2.SU2
- net USART3_RX: now also P1.SD3; no longer P2.SD3
- net USART3_TX: now also P1.SU3; no longer P2.SU3
- net USART5_RX: now also P1.SD12; no longer P2.SD5
- net USART5_TX: now also P1.SU12; no longer P2.SU5
- net USART6_RX: now also P1.SD13; no longer P2.SD1
- net USART6_TX: now also P1.SU13; no longer P2.SU1
- net VDD: now also C37.2, C44.2, C45.1, C6.2, FB1.1, P1.VDD1, P1.VDD10, P1.VDD11, P1.VDD12, P1.VDD13, P1.VDD2, P1.VDD3, P1.VDD4, P1.VDD5, P1.VDD6, R6.2, R7.1, R8.1, R9.2, U2.DVDDIO, U3.VCC, U6.EN, U6.VIN; no longer C5.1, FB1.2, P2.VDD1, P2.VDD2, P2.VDD3, P2.VDD4, P2.VDD5, P2.VDD6, P2.VDD7, P2.VDD8
- net VDDA: now also C2.2, C3.+, C4.2, C5.+, FB1.2; no longer C1.1, C2.+, C3.1, C4.+, FB1.1
Other:
- note added: "3"
- note added: "Audio Jack For External Input"
- note added: "B"
- note added: "H07R8_Backened"
- note added: "H07R8_Frontened"
- note added: "Power Amplifier 12V External Input"
- note added: "Speaker Left"
- note added: "Speaker Right"
- note added: "VDD\\\VDDA Coupling"
- note removed: "BOOT"
- note removed: "C:/Users/Admin/Desktop/logodraft.bmp"
- note removed: "H07R8_Backend"
- note removed: "H07R8_Frontend"
- note removed: "Muhammad Awais"
- note removed: "VDD=3.3 Volts"
- note removed: "VDD\VDDA Coupling"
